File: PCB board design/Review_day_PCB/Review_PCD_1.3.brd (EAGLE design)
At the start: 160 x 100 mm, 9 parts, among them IC1 ATMEGA168-20P

Commit message: rev.1.3
Routing:
- net 0: track 162.6 -> 260.4 mm
- net N$2: track 21.6 -> 66.2 mm, vias 0 -> 1
- net N$15: track 87.9 -> 121.0 mm
- net N$14: track 37.9 -> 67.4 mm
- net N$1: track 228.3 -> 248.1 mm
- net N$13: track 36.4 -> 55.1 mm
Changed lines of the file:
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@@
 <wire x1="83.82" y1="52.07" x2="83.82" y2="30.3276" width="0.1524" layer="16"/>
 <contactref element="JP1" pad="2"/>
-<wire x1="128.27" y1="59.69" x2="97.79" y2="74.76" width="0" layer="19" extent="1-1"/>
+<wire x1="97.6884" y1="73.6092" x2="97.6884" y2="74.676" width="0.1524" layer="16"/>
+<wire x1="86.4108" y1="62.3316" x2="97.6884" y2="73.6092" width="0.1524" layer="16"/>
+<wire x1="86.4108" y1="59.7408" x2="86.4108" y2="62.3316" width="0.1524" layer="16"/>
+<wire x1="97.6884" y1="74.676" x2="97.79" y2="74.76" width="0.1524" layer="16"/>
+<wire x1="86.4108" y1="59.7408" x2="86.36" y2="59.69" width="0.1524" layer="16"/>
 </signal>
 <signal name="N$2">
@@
 <contactref element="R1" pad="1"/>
 <wire x1="59.436" y1="61.2648" x2="50.9016" y2="61.2648" width="0.1524" layer="1"/>
-<wire x1="68.58" y1="52.1208" x2="59.436" y2="61.2648" width="0.1524" layer="1"/>
+<wire x1="68.58" y1="52.1208" x2="67.056" y2="53.6448" width="0.1524" layer="1"/>
+<wire x1="67.056" y1="53.6448" x2="59.436" y2="61.2648" width="0.1524" layer="1"/>
 <wire x1="50.9016" y1="61.2648" x2="50.8" y2="61.29" width="0.1524" layer="1"/>
 <wire x1="68.58" y1="52.1208" x2="68.58" y2="52.07" width="0.1524" layer="1"/>
 <contactref element="JP1" pad="5"/>
-<wire x1="68.58" y1="52.07" x2="97.79" y2="85.26" width="0" layer="19" extent="1-1"/>
+<wire x1="97.2312" y1="85.1916" x2="97.6884" y2="85.1916" width="0.1524" layer="16"/>
+<wire x1="72.39" y1="60.3504" x2="97.2312" y2="85.1916" width="0.1524" layer="16"/>
+<wire x1="72.39" y1="58.9788" x2="72.39" y2="60.3504" width="0.1524" layer="1"/>
+<wire x1="67.056" y1="53.6448" x2="72.39" y2="58.9788" width="0.1524" layer="1"/>
+<wire x1="97.6884" y1="85.1916" x2="97.79" y2="85.26" width="0.1524" layer="16"/>
+<via x="72.39" y="60.3504" extent="1-16" drill="0.35"/>
 </signal>
 <signal name="0">
@@
 <contactref element="DIS1" pad="5"/>
 <contactref element="JP1" pad="6"/>
-<wire x1="128.27" y1="52.07" x2="97.79" y2="88.76" width="0" layer="19" extent="1-1"/>
-<wire x1="50.8" y1="51.13" x2="50.9016" y2="51.054" width="0" layer="19" extent="1-1"/>
-<wire x1="50.7492" y1="51.2064" x2="50.8" y2="51.13" width="0" layer="19" extent="1-1"/>
-<wire x1="21.21" y1="24.13" x2="51.175" y2="47.735" width="0" layer="19" extent="1-1"/>
+<wire x1="50.7492" y1="51.2064" x2="50.8" y2="51.13" width="0.1524" layer="1"/>
+<wire x1="50.9016" y1="51.054" x2="50.8" y2="51.13" width="0.1524" layer="1"/>
+<wire x1="42.0624" y1="48.768" x2="50.292" y2="48.768" width="0.1524" layer="1"/>
+<wire x1="18.288" y1="24.9936" x2="42.0624" y2="48.768" width="0.1524" layer="1"/>
+<wire x1="18.288" y1="23.3172" x2="18.288" y2="24.9936" width="0.1524" layer="1"/>
+<wire x1="18.4404" y1="23.1648" x2="18.288" y2="23.3172" width="0.1524" layer="1"/>
+<wire x1="20.2692" y1="23.1648" x2="18.4404" y2="23.1648" width="0.1524" layer="1"/>
+<wire x1="21.1836" y1="24.0792" x2="20.2692" y2="23.1648" width="0.1524" layer="1"/>
+<wire x1="50.292" y1="48.768" x2="50.425" y2="48.785" width="0.1524" layer="1"/>
+<wire x1="21.1836" y1="24.0792" x2="21.21" y2="24.13" width="0.1524" layer="1"/>
+<wire x1="97.8408" y1="87.1728" x2="97.8408" y2="88.6968" width="0.1524" layer="1"/>
+<wire x1="127.254" y1="57.7596" x2="97.8408" y2="87.1728" width="0.1524" layer="1"/>
+<wire x1="127.254" y1="56.6928" x2="127.254" y2="57.7596" width="0.1524" layer="1"/>
+<wire x1="128.3208" y1="55.626" x2="127.254" y2="56.6928" width="0.1524" layer="1"/>
+<wire x1="128.778" y1="55.626" x2="128.3208" y2="55.626" width="0.1524" layer="1"/>
+<wire x1="129.3876" y1="55.0164" x2="128.778" y2="55.626" width="0.1524" layer="1"/>
+<wire x1="129.3876" y1="53.1876" x2="129.3876" y2="55.0164" width="0.1524" layer="1"/>
+<wire x1="128.27" y1="52.07" x2="129.3876" y2="53.1876" width="0.1524" layer="1"/>
+<wire x1="97.8408" y1="88.6968" x2="97.79" y2="88.76" width="0.1524" layer="1"/>
 </signal>
 <signal name="N$3">
@@
 <wire x1="127.5588" y1="57.7596" x2="93.8784" y2="57.7596" width="0.1524" layer="16"/>
 <wire x1="128.1684" y1="57.15" x2="127.5588" y2="57.7596" width="0.1524" layer="16"/>
-<wire x1="91.44" y1="59.5884" x2="91.44" y2="59.69" width="0.1524" layer="16"/>
 <wire x1="128.1684" y1="57.15" x2="128.27" y2="57.15" width="0.1524" layer="16"/>
 <contactref element="JP1" pad="3"/>
-<wire x1="91.44" y1="59.69" x2="97.79" y2="78.26" width="0" layer="19" extent="1-1"/>
+<wire x1="97.8408" y1="76.6572" x2="97.8408" y2="78.1812" width="0.1524" layer="16"/>
+<wire x1="99.2124" y1="75.2856" x2="97.8408" y2="76.6572" width="0.1524" layer="16"/>
+<wire x1="99.2124" y1="74.2188" x2="99.2124" y2="75.2856" width="0.1524" layer="16"/>
+<wire x1="97.6884" y1="72.6948" x2="99.2124" y2="74.2188" width="0.1524" layer="16"/>
+<wire x1="97.2312" y1="72.6948" x2="97.6884" y2="72.6948" width="0.1524" layer="16"/>
+<wire x1="87.9348" y1="63.3984" x2="97.2312" y2="72.6948" width="0.1524" layer="16"/>
+<wire x1="87.9348" y1="58.674" x2="87.9348" y2="63.3984" width="0.1524" layer="16"/>
+<wire x1="88.5444" y1="58.0644" x2="87.9348" y2="58.674" width="0.1524" layer="16"/>
+<wire x1="89.916" y1="58.0644" x2="88.5444" y2="58.0644" width="0.1524" layer="16"/>
+<wire x1="91.44" y1="59.5884" x2="89.916" y2="58.0644" width="0.1524" layer="16"/>
+<wire x1="97.8408" y1="78.1812" x2="97.79" y2="78.26" width="0.1524" layer="16"/>
+<wire x1="91.44" y1="59.5884" x2="91.44" y2="59.69" width="0.1524" layer="16"/>
 </signal>
 <signal name="N$11">
@@
 <wire x1="94.6404" y1="59.5884" x2="94.0308" y2="59.5884" width="0.1524" layer="1"/>
 <wire x1="99.5172" y1="54.7116" x2="94.6404" y2="59.5884" width="0.1524" layer="1"/>
-<wire x1="128.1684" y1="54.7116" x2="99.5172" y2="54.7116" width="0.1524" layer="1"/>
+<wire x1="128.1684" y1="54.7116" x2="102.87" y2="54.7116" width="0.1524" layer="1"/>
+<wire x1="102.87" y1="54.7116" x2="99.5172" y2="54.7116" width="0.1524" layer="1"/>
 <wire x1="94.0308" y1="59.5884" x2="93.98" y2="59.69" width="0.1524" layer="1"/>
 <wire x1="128.1684" y1="54.7116" x2="128.27" y2="54.61" width="0.1524" layer="1"/>
-<wire x1="93.98" y1="59.69" x2="97.79" y2="71.26" width="0" layer="19" extent="1-1"/>
+<wire x1="97.8408" y1="65.8368" x2="97.8408" y2="71.1708" width="0.1524" layer="1"/>
+<wire x1="102.87" y1="60.8076" x2="97.8408" y2="65.8368" width="0.1524" layer="1"/>
+<wire x1="102.87" y1="54.7116" x2="102.87" y2="60.8076" width="0.1524" layer="1"/>
+<wire x1="97.8408" y1="71.1708" x2="97.79" y2="71.26" width="0.1524" layer="1"/>
 </signal>
 <signal name="N$15">
@@
 <wire x1="96.4692" y1="59.7408" x2="96.52" y2="59.69" width="0.1524" layer="1"/>
 <wire x1="21.336" y1="87.63" x2="21.21" y2="87.63" width="0.1524" layer="1"/>
-<wire x1="96.52" y1="59.69" x2="97.79" y2="81.76" width="0" layer="19" extent="1-1"/>
+<wire x1="97.6884" y1="80.1624" x2="97.6884" y2="81.6864" width="0.1524" layer="1"/>
+<wire x1="96.4692" y1="78.9432" x2="97.6884" y2="80.1624" width="0.1524" layer="1"/>
+<wire x1="96.4692" y1="66.7512" x2="96.4692" y2="78.9432" width="0.1524" layer="1"/>
+<wire x1="102.5652" y1="60.6552" x2="96.4692" y2="66.7512" width="0.1524" layer="1"/>
+<wire x1="102.5652" y1="58.674" x2="102.5652" y2="60.6552" width="0.1524" layer="1"/>
+<wire x1="101.9556" y1="58.0644" x2="102.5652" y2="58.674" width="0.1524" layer="1"/>
+<wire x1="98.1456" y1="58.0644" x2="101.9556" y2="58.0644" width="0.1524" layer="1"/>
+<wire x1="96.52" y1="59.69" x2="98.1456" y2="58.0644" width="0.1524" layer="1"/>
+<wire x1="97.6884" y1="81.6864" x2="97.79" y2="81.76" width="0.1524" layer="1"/>
 </signal>
 </signals>
