File: PCB board design/Review_day_PCB/Review_PCD_1.4.brd (EAGLE design)
At the start: 160 x 100 mm, 9 parts, among them U1 ATMEGA328P_VQFNVQFN

Commit message: changed to atmega328p
Parts:
- Q1: value (none) -> 16 MHz
- R1, R3: value (none) -> 10 kOhm
- R2: value (none) -> 1 kOhm
Connections:
- net N$1 renamed VCC
- removed net 0: DIS1.18, DIS1.5, G1.-, JP1.6, Q1.1, Q1.3, R3.1, U$1.4, U1.5, U1.6
- new net GND: DIS1.10, DIS1.18, DIS1.5, DIS1.7, DIS1.8, DIS1.9, G1.-, JP1.6, Q1.1, Q1.3, R3.1, U$1.4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
Routing:
- net GND: track 0.00 -> 254.9 mm
- net 0: track 254.9 -> 0.00 mm
