File: PCB board design/Review_day_PCB/Review_PCD_1.4.sch (EAGLE design)
At the start: 9 parts, among them U1 ATMEGA328P_VQFNVQFN

Commit message: changed to atmega328p
Parts:
- Q1: value (none) -> 16 MHz
- R1: value (none) -> 10 kOhm; R1 10 kOhm -> (none)
- R2: value (none) -> 1 kOhm
- R3: value (none) -> 10 kOhm
Connections:
- net N$1 renamed VCC
- removed net 0: DIS1.C, DIS1.R/W, G1.-, JP1.6, Q1.1, Q1.2, R3.1, U$1.GND, U1.PB6(XTAL1/TOSC1), U1.PB7(XTAL2/TOSC2)
- new net GND: DIS1.C, DIS1.D0, DIS1.D1, DIS1.D2, DIS1.D3, DIS1.R/W, G1.-, JP1.6, Q1.1, Q1.2, R3.1, U$1.GND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
