File: PCB board design/Review_day_PCB/Review_PCD_1.5.sch (EAGLE design)
At the start: 9 parts, among them Q1 16 MHz, U1 ATMEGA328P_VQFNVQFN

Commit message: all correct components and no errors
Parts:
- removed DIS1: EA_DIP, display-lcd:EA_DIP
- removed U$1: ULTRASONIC-HC-SR04, diy-modules:ULTRASONIC-HC-SR04
- added JP2: Pinout to UltraSonic sensor, adafruit:PINHD-1X6B
- added JP3: Pinout to LCD, adafruit:PINHD-1X18
- added Q2: 2N7000, m-pad-2.1:2N7000KL/BS170KL
- JP1: value (none) -> Programmable Pinout
- renumbered G1 to 5V
Connections:
- removed net 0: DIS1.D0, DIS1.D1, DIS1.D2, DIS1.D3
- removed net GND: 5V.-, DIS1.C, DIS1.R/W, JP1.6, Q1.1, Q1.2, R3.1, U$1.GND, U1.PB6(XTAL1/TOSC1), U1.PB7(XTAL2/TOSC2)
- removed net N$11: DIS1.VEE, R3.2
- removed net N$13: JP1.1, U$1.ECHO, U1.PB4(MISO)
- removed net N$14: JP1.3, U$1.TRIG, U1.PB5(SCK)
- removed net N$15: DIS1.D7, JP1.4, U1.PB3(MOSI/OC2)
- removed net N$5: DIS1.RS, U1.PD6(AIN0)
- removed net N$6: DIS1.E, U1.PD7(AIN1)
- removed net N$7: DIS1.D4, U1.PB0(ICP)
- removed net N$8: DIS1.D5, U1.PB1(OC1A)
- removed net N$9: DIS1.D6, U1.PB2(SS/OC1B)
- removed net VCC: 5V.+, DIS1.A, DIS1.VDD, DIS1.VSS, JP1.2, R1.2, U$1.VCC, U1.AREF, U1.AVCC, U1.PC0(ADC0), U1.VCC
- new net C: 5V.-, JP1.6, JP3.18, Q1.1, Q1.2, Q2.S, R3.1, U1.PB6(XTAL1/TOSC1), U1.PB7(XTAL2/TOSC2)
- new net D4: JP3.11, U1.PB0(ICP)
- new net D5: JP3.12, U1.PB1(OC1A)
- new net D6: JP3.13, U1.PB2(SS/OC1B)
- new net D7: JP1.4, JP3.14, U1.PB3(MOSI/OC2)
- new net E: JP3.6, U1.PD7(AIN1)
- new net ECHO: JP1.1, JP2.3, U1.PB4(MISO)
- new net N$1: Q2.G, R2.2
- new net RS: JP3.4, U1.PD6(AIN0)
- new net TRIG: JP1.3, JP2.2, U1.PB5(SCK)
- new net VEE: JP3.3, R3.2
- new net VSS: 5V.+, JP1.2, JP2.1, JP3.1, JP3.17, JP3.2, Q2.D, R1.2, U1.AREF, U1.AVCC, U1.PC0(ADC0), U1.VCC
- net N$4: now also JP2.4, JP2.5, JP2.6; no longer R2.2
Other:
- note added: "A"
- note added: "D0"
- note added: "D1"
- note added: "D2"
- note added: "D3"
- note added: "NC"
- note added: "RW"
- note added: "VDD"
- note removed: "2n7000 MOSFET Gate"
