File: PCB board design/Review_day_PCB/Review_PCD_1.8.sch (EAGLE design)
At the start: 10 parts, among them Q1 16 MHz, Q2 2N7000, U1 ATMEGA328P_VQFNVQFN

Commit message: navid saved the day
Parts:
- removed Q1: 16 MHz, crystal-geyer_V1_0:KX-4
- added C1, C2: 22pF, SparkFun-Capacitors:22PF-PTH-2.54MM-200V-5%
- added Y1: 16MHz, SparkFun-Clocks:CRYSTAL-16MHZPTH-HC49US
Connections:
- new net 0: C1.1, C2.1, JP1.6, POWER.2, POWER.3
- new net N$4: C1.2, U1.PB6(XTAL1/TOSC1), Y1.2
- new net N$5: C2.2, U1.PB7(XTAL2/TOSC2), Y1.1
- new net N$6: JP2.4, JP2.5, JP2.6, JP3.18, Q2.S, R3.1
- net C: no longer JP1.6, JP2.4, JP2.5, JP2.6, JP3.18, POWER.2, POWER.3, Q1.1, Q1.2, Q2.S, R3.1, U1.PB6(XTAL1/TOSC1), U1.PB7(XTAL2/TOSC2)
Other:
- moved on the sheet: JP1
